File: Electronique/Kicad/Afficheur-Led [1:2]/Afficheur-Led-1:2.sch (KiCad schematic (older format))
At the start: 60 parts, among them J1 Screw_Terminal_01x02, J10 Screw_Terminal_01x02, J11 Screw_Terminal_01x02, J2 Screw_Terminal_01x02, J3 Screw_Terminal_01x02, J4 Screw_Terminal_01x02, J5 Screw_Terminal_01x02, J6 Screw_Terminal_01x02, J7 Screw_Terminal_01x02, J8 Screw_Terminal_01x02, J9 Screw_Terminal_01x02, Q1 PN2222A, Q10 PN2222A, Q11 PN2222A, Q12 PN2222A, Q13 PN2222A, Q14 PN2222A, Q15 PN2222A, Q16 PN2222A, Q17 PN2222A, Q18 PN2222A, Q19 PN2222A, Q2 PN2222A, Q20 PN2222A, Q3 PN2222A, Q4 PN2222A, Q5 PN2222A, Q6 PN2222A, Q7 PN2222A, Q8 PN2222A, Q9 PN2222A, U1 Arduino_pro_Mini_[A], U2 LM7805_TO220, U3 RF_Transmitter_433Mhz_OPEN-SM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, U4 74HC595, U5 74HC595

Commit message: up
Parts:
- removed C1: 0,3uF, Capacitors_THT:C_Disc_D5.0mm_W2.5mm_P5.00mm, symbol C
- removed C2: 0,1uF, Capacitors_THT:C_Disc_D5.0mm_W2.5mm_P5.00mm, symbol C
- removed J10, J11, J2, J3, J4, J5, J6, J7, J8, J9: Screw_Terminal_01x02, Connectors_Terminal_Blocks:TerminalBlock_Pheonix_MPT-2.54mm_2pol, symbol Screw_Terminal_01x02
- removed U2: LM7805_TO220, TO_SOT_Packages_THT:TO-220-3_Vertical, symbol LM7805_TO220
- added J2, J3, J4, J5: Conn_01x05, Pin_Headers:Pin_Header_Angled_1x05_Pitch2.54mm, symbol Conn_01x05
- added U2: 74HC595, Housings_DIP:DIP-16_W7.62mm, symbol 74HC595
Connections:
- net labels removed: +12V
- wire segments 207 -> 230
