File: Electronique/Kicad/Afficheur-Led [2:2]/Afficheur-Led-2:2.sch (KiCad schematic (older format))
At the start: 53 parts, among them U1 Arduino_pro_Mini_[A], U2 LM7805_TO220, U3 4051, U4 4051, U5 LM317_TO3, U6 RF-440mhz-Emitter

Commit message: up
Connections:
- net at U1.11 (D2): no longer U6.~ (VCC)
- net at U1.12 (D3): now also U3.11 (A), U4.11 (A)
- net at U1.13 (D4): now also U3.10 (B), U4.10 (B)
- net at U1.14 (D5): now also U3.9 (C), U4.9 (C)
- net at U1.17 (D8): now also R6.2
- net at U1.18 (D9): now also R10.2
- net at U1.23 (A3): no longer R10.2
- net at U1.24 (A2): no longer R6.2
- net at R18.2: now also U1.29 (D11); no longer U1.31 (A5)
- net at R14.2: now also U1.30 (D10); no longer U1.32 (A4)
- now unconnected: U1.28 (D12)
Changed lines of the file:
@@
 LIBS:contrib
 LIBS:valves
-LIBS:Afficheur-Led-2:2
 LIBS:Afficheur-Led-2:2-cache
 EELAYER 25 0
@@
 Connection ~ 3050 5600
 Wire Wire Line
-	1900 2350 1900 3500
+	1900 2350 1900 3200
+Wire Wire Line
+	1900 3200 1900 3500
 Connection ~ 1900 2350
 Connection ~ 3050 6600
@@
 	1300 5650 1450 5650
 Wire Wire Line
-	2200 4050 2200 3500
+	2200 4050 2200 3800
+Wire Wire Line
+	2200 3800 2200 3500
 Connection ~ 3050 5500
 Connection ~ 3050 5400
@@
 Connection ~ 2200 3800
 Wire Wire Line
-	1900 3800 2500 3800
+	1900 3800 2200 3800
+Wire Wire Line
+	2200 3800 2500 3800
 Connection ~ 1900 3200
 Connection ~ 1100 2350
@@
 Connection ~ 5700 6200
 Wire Wire Line
-	5700 5850 5700 6200
+	5700 5850 5700 6050
+Wire Wire Line
+	5700 6050 5700 6200
 Wire Wire Line
 	5700 5850 6400 5850
@@
 Connection ~ 5700 7600
 Wire Wire Line
-	5700 7250 5700 7600
+	5700 7250 5700 7450
+Wire Wire Line
+	5700 7450 5700 7600
 Wire Wire Line
 	5700 7250 6400 7250
@@
 Connection ~ 5850 4850
 Wire Wire Line
-	3050 6100 4050 6100
-Wire Wire Line
-	3050 6200 4150 6200
-Wire Wire Line
-	4150 6200 4150 8050
-Wire Wire Line
-	3050 6300 4250 6300
-Wire Wire Line
-	4250 6300 4250 8150
-Connection ~ 4250 6300
-Connection ~ 4150 6200
-Connection ~ 4050 6100
-Wire Wire Line
-	4450 7450 5700 7450
-Wire Wire Line
-	4450 6050 5700 6050
-Wire Wire Line
-	4050 6100 4050 7950
+	3050 5400 4050 5950
+Wire Wire Line
+	3050 5500 4150 6100
+Wire Wire Line
+	4150 6100 4150 8050
+Wire Wire Line
+	3050 5600 4250 6250
+Wire Wire Line
+	4250 6250 4250 8150
+Connection ~ 4250 6250
+Connection ~ 4150 6100
+Connection ~ 4050 5950
+Wire Wire Line
+	4450 7450 5000 7450
+Wire Wire Line
+	5000 7450 5700 7450
+Wire Wire Line
+	4450 6050 5000 6050
+Wire Wire Line
+	5000 6050 5700 6050
+Wire Wire Line
+	4050 5950 4050 7950
 Wire Wire Line
 	4050 7950 6750 7950
 Wire Wire Line
-	6750 7950 6750 5950
+	6750 7950 6750 7350
+Wire Wire Line
+	6750 7350 6750 5950
 Wire Wire Line
 	6750 7350 6400 7350
@@
 	6400 7450 6650 7450
 Wire Wire Line
-	6650 6050 6650 8050
+	6650 6050 6650 7450
+Wire Wire Line
+	6650 7450 6650 8050
 Wire Wire Line
 	6650 8050 4150 8050
@@
 	4250 8150 6550 8150
 Wire Wire Line
-	6550 8150 6550 6150
+	6550 8150 6550 7550
+Wire Wire Line
+	6550 7550 6550 6150
 Wire Wire Line
 	6550 7550 6400 7550
@@
 Connection ~ 6750 7350
 Wire Wire Line
-	3050 6600 3700 6600
-Wire Wire Line
-	3700 6600 3700 4950
+	3050 6600 3700 6050
+Wire Wire Line
+	3700 6050 3700 4950
 Wire Wire Line
 	3700 4950 5000 4950
 Wire Wire Line
-	3050 6700 5000 6700
-Wire Wire Line
-	5000 6700 5000 6350
-Wire Wire Line
-	3650 6800 3650 8250
-Wire Wire Line
-	3650 6800 3050 6800
-Wire Wire Line
-	3050 6900 3550 6900
-Wire Wire Line
-	3550 6900 3550 8350
-Wire Wire Line
-	3450 7100 3450 8450
-Wire Wire Line
-	3450 7100 3050 7100
-Wire Wire Line
-	3050 7200 3350 7200
-Wire Wire Line
-	3350 7200 3350 8550
+	3050 6700 5000 6850
+Wire Wire Line
+	5000 6850 5000 6350
+Wire Wire Line
+	3650 6250 3650 8250
+Wire Wire Line
+	3650 6250 3050 5900
+Wire Wire Line
+	3050 6000 3550 6300
+Wire Wire Line
+	3550 6300 3550 8350
+Wire Wire Line
+	3450 6350 3450 8450
+Wire Wire Line
+	3450 6350 3050 6100
+Wire Wire Line
+	3050 6200 3350 6400
+Wire Wire Line
+	3350 6400 3350 8550
 Connection ~ 9050 3500
 Connection ~ 14300 3500
@@
 	7250 8550 7250 7850
 Wire Wire Line
-	1100 1900 2500 1900
-Wire Wire Line
-	3100 1900 5100 1900
-Wire Wire Line
-	2800 1350 2800 1600
+	1100 1900 2400 1900
+Wire Wire Line
+	2400 1900 2500 1900
+Wire Wire Line
+	3100 1900 3300 1900
+Wire Wire Line
+	3300 1900 3650 1900
+Wire Wire Line
+	3650 1900 5100 1900
+Wire Wire Line
+	2800 1350 2800 1450
+Wire Wire Line
+	2800 1450 2800 1600
 Wire Wire Line
 	2800 1450 3300 1450
@@
 	2400 1300 2400 1050
 Wire Wire Line
-	800  1050 3850 1050
+	800  1050 2400 1050
+Wire Wire Line
+	2400 1050 2800 1050
+Wire Wire Line
+	2800 1050 3300 1050
+Wire Wire Line
+	3300 1050 3650 1050
+Wire Wire Line
+	3650 1050 3850 1050
 Connection ~ 2800 1350
 Connection ~ 3300 1750
@@
 Connection ~ 2200 4050
 Wire Wire Line
-	5850 6250 5850 4400
+	5850 6250 5850 4850
+Wire Wire Line
+	5850 4850 5850 4400
 Wire Wire Line
 	2500 3200 4650 3200
 Wire Wire Line
-	5850 4400 1300 4400
+	5850 4400 4650 4400
+Wire Wire Line
+	4650 4400 1300 4400
 Connection ~ 4650 3200
 Wire Wire Line
@@
 	6200 2200 3250 2200
 Wire Wire Line
-	3250 2200 3250 5300
-Wire Wire Line
-	3250 5300 3050 5300
+	3250 2200 3250 4900
 Wire Wire Line
 	5100 1600 4900 1600
@@
 	4900 1050 4550 1050
 Wire Wire Line
-	800  4050 4450 4050
-Wire Wire Line
-	4650 2550 4650 4400
+	800  4050 1050 4050
+Wire Wire Line
+	1050 4050 2200 4050
+Wire Wire Line
+	2200 4050 4450 4050
+Wire Wire Line
+	4650 2550 4650 3200
+Wire Wire Line
+	4650 3200 4650 4400
 Wire Wire Line
 	1100 2350 1100 1900
@@
 	9050 3500 9050 4100
 Wire Wire Line
-	9050 4100 15750 4100
+	9050 4100 10800 4100
+Wire Wire Line
+	10800 4100 12550 4100
+Wire Wire Line
+	12550 4100 14300 4100
+Wire Wire Line
+	14300 4100 15750 4100
 Wire Wire Line
 	9050 5150 9050 5700
 Wire Wire Line
-	9050 5700 15750 5700
+	9050 5700 10800 5700
+Wire Wire Line
+	10800 5700 12550 5700
+Wire Wire Line
+	12550 5700 14300 5700
+Wire Wire Line
+	14300 5700 15750 5700
 Wire Wire Line
 	9050 6750 9050 7350
 Wire Wire Line
-	9050 7350 15750 7350
+	9050 7350 10800 7350
+Wire Wire Line
+	10800 7350 12550 7350
+Wire Wire Line
+	12550 7350 14300 7350
+Wire Wire Line
+	14300 7350 15750 7350
 Wire Wire Line
 	9050 8400 9050 9000
 Wire Wire Line
-	9050 9000 15750 9000
-Wire Wire Line
-	15750 9000 15750 2550
+	9050 9000 10800 9000
+Wire Wire Line
+	10800 9000 12550 9000
+Wire Wire Line
+	12550 9000 14300 9000
+Wire Wire Line
+	14300 9000 15750 9000
+Wire Wire Line
+	15750 9000 15750 4100
+Wire Wire Line
+	15750 4100 15750 2550
 Connection ~ 15750 4100
 Wire Wire Line
@@
 $EndComp
 Wire Wire Line
-	4450 4050 4450 7450
+	4450 4050 4450 6050
+Wire Wire Line
+	4450 6050 4450 7450
 Connection ~ 4450 6050
 $Comp
@@
 	8350 2100 8350 2250
 Wire Wire Line
-	8350 2250 13300 2250
+	8350 2250 9900 2250
+Wire Wire Line
+	9900 2250 11750 2250
+Wire Wire Line
+	11750 2250 13300 2250
 Wire Wire Line
 	9900 2250 9900 2100
